Commit message: 24

File: src/rebot_description/urdf/reBot_B601_DM_with_gripper.urdf (robot description, URDF)
Before this commit: robot reBot_B601_DM_with_gripper, 10 links, 9 joints
Links:
- link base_link: geometry collision mesh filename=package://rebot_description/urdf/meshes_b601_gripper/base_l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; visual mesh filename=package://rebot_description/urdf/meshes_b601_gripper/base_l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
- link gripper_left: geometry collision mesh filename=package://rebot_description/urdf/meshes_b601_gripper/grippe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; visual mesh filename=package://rebot_description/urdf/meshes_b601_gripper/grippe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
- link gripper_link: geometry collision mesh filename=package://rebot_description/urdf/meshes_b601_gripper/grippe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; visual mesh filename=package://rebot_description/urdf/meshes_b601_gripper/grippe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
- link gripper_right: geometry collision mesh filename=package://rebot_description/urdf/meshes_b601_gripper/grippe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; visual mesh filename=package://rebot_description/urdf/meshes_b601_gripper/grippe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
- link link1: geometry collision mesh filename=package://rebot_description/urdf/meshes_b601_gripper/link1.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; visual mesh filename=package://rebot_description/urdf/meshes_b601_gripper/link1.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
- link link2: geometry collision mesh filename=package://rebot_description/urdf/meshes_b601_gripper/link2.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; visual mesh filename=package://rebot_description/urdf/meshes_b601_gripper/link2.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
- link link3: geometry collision mesh filename=package://rebot_description/urdf/meshes_b601_gripper/link3.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; visual mesh filename=package://rebot_description/urdf/meshes_b601_gripper/link3.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
- link link4: geometry collision mesh filename=package://rebot_description/urdf/meshes_b601_gripper/link4.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; visual mesh filename=package://rebot_description/urdf/meshes_b601_gripper/link4.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
- link link5: geometry collision mesh filename=package://rebot_description/urdf/meshes_b601_gripper/link5.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; visual mesh filename=package://rebot_description/urdf/meshes_b601_gripper/link5.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
- link link6: geometry collision mesh filename=package://rebot_description/urdf/meshes_b601_gripper/link6.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; visual mesh filename=package://rebot_description/urdf/meshes_b601_gripper/link6.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
